File: power_tester.brd (EAGLE design)
At the start: 85.4 x 100 mm, 104 parts, among them IC1 MEGA8-AI, IC2 7805DT, IC3 LMV324M, Q1 BC547, Q2 IRF3704TO252, Q3 IRF3704TO252, Q4 IRF3704TO252, T1 BC547, T2 BC547, T3 BC547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

Commit message: change
change
Connections:
- net CA1: now also IC1.23; no longer IC1.22
- net CA2: now also IC1.24; no longer IC1.19
- net N$58: now also IC1.22; no longer IC1.24
- net N$59: now also IC1.19; no longer IC1.23
Routing:
- net N$59: track 43.9 -> 56.1 mm
- net CA1: track 74.7 -> 81.4 mm, vias 0 -> 2
- net N$58: track 40.2 -> 46.1 mm
- net CA2: track 63.1 -> 68.4 mm, vias 0 -> 2
