File: power_tester.sch (EAGLE design)
At the start: 104 parts, among them IC1 MEGA8-AI, IC2 7805DT, IC3 LMV324M, Q1 BC547, Q2 IRF3704TO252, Q3 IRF3704TO252, Q4 IRF3704TO252, T1 BC547, T2 BC547, T3 BC547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

Commit message: change
change
Connections:
- net CA1: now also IC1.PC0(ADC0); no longer IC1.ADC7
- net CA2: now also IC1.PC1(ADC1); no longer IC1.ADC6
- net N$58: now also IC1.ADC7; no longer IC1.PC1(ADC1)
- net N$59: now also IC1.ADC6; no longer IC1.PC0(ADC0)
Changed lines of the file:
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@@
 </segment>
 <segment>
-<pinref part="IC1" gate="G$1" pin="ADC6"/>
-<wire x1="-111.76" y1="12.7" x2="-106.68" y2="12.7" width="0.1524" layer="91"/>
+<pinref part="IC1" gate="G$1" pin="PC1(ADC1)"/>
+<wire x1="-111.76" y1="25.4" x2="-121.92" y2="25.4" width="0.1524" layer="91"/>
+<wire x1="-121.92" y1="25.4" x2="-121.92" y2="7.62" width="0.1524" layer="91"/>
+<wire x1="-106.68" y1="7.62" x2="-121.92" y2="7.62" width="0.1524" layer="91"/>
 </segment>
 </net>
@@
 </segment>
 <segment>
-<pinref part="IC1" gate="G$1" pin="ADC7"/>
-<wire x1="-111.76" y1="10.16" x2="-106.68" y2="10.16" width="0.1524" layer="91"/>
+<wire x1="-106.68" y1="-15.24" x2="-124.46" y2="-15.24" width="0.1524" layer="91"/>
+<wire x1="-124.46" y1="-15.24" x2="-124.46" y2="27.94" width="0.1524" layer="91"/>
+<pinref part="IC1" gate="G$1" pin="PC0(ADC0)"/>
+<wire x1="-124.46" y1="27.94" x2="-111.76" y2="27.94" width="0.1524" layer="91"/>
 </segment>
 </net>
@@
 </segment>
 </net>
-<net name="N$58" class="0">
-<segment>
-<pinref part="R50" gate="G$1" pin="1"/>
-<wire x1="-101.6" y1="25.4" x2="-101.6" y2="-7.62" width="0.1524" layer="91"/>
-<pinref part="IC1" gate="G$1" pin="PC1(ADC1)"/>
-<wire x1="-101.6" y1="25.4" x2="-111.76" y2="25.4" width="0.1524" layer="91"/>
-</segment>
-</net>
-<net name="N$59" class="0">
-<segment>
-<pinref part="IC1" gate="G$1" pin="PC0(ADC0)"/>
-<wire x1="-111.76" y1="27.94" x2="-111.76" y2="48.26" width="0.1524" layer="91"/>
-<pinref part="R51" gate="G$1" pin="2"/>
-<wire x1="-109.22" y1="48.26" x2="-111.76" y2="48.26" width="0.1524" layer="91"/>
-</segment>
-</net>
 <net name="N$60" class="0">
 <segment>
@@
 </segment>
 </net>
+<net name="N$59" class="0">
+<segment>
+<pinref part="R51" gate="G$1" pin="2"/>
+<wire x1="-109.22" y1="48.26" x2="-127" y2="48.26" width="0.1524" layer="91"/>
+<wire x1="-127" y1="48.26" x2="-127" y2="12.7" width="0.1524" layer="91"/>
+<pinref part="IC1" gate="G$1" pin="ADC6"/>
+<wire x1="-127" y1="12.7" x2="-111.76" y2="12.7" width="0.1524" layer="91"/>
+</segment>
+</net>
+<net name="N$58" class="0">
+<segment>
+<pinref part="IC1" gate="G$1" pin="ADC7"/>
+<wire x1="-111.76" y1="10.16" x2="-101.6" y2="10.16" width="0.1524" layer="91"/>
+<pinref part="R50" gate="G$1" pin="1"/>
+<wire x1="-101.6" y1="10.16" x2="-101.6" y2="-7.62" width="0.1524" layer="91"/>
+</segment>
+</net>
